File: hardware/module_controller/_autosave-ModuleController.kicad_pcb (KiCad board)
At the start: 2 copper layers, 60 x 90 mm, 24 parts, among them J1 JST05_StepperMotor, J6 Conn_02x08_Top_Bottom, U1 ULN2003, U2 A1101ELHL, U3 SN75176AP, U4 ATmega8A-A, Y1 16MHz

Commit message: update schematics
Parts:
- F1: value Polyfuse 10ma/20mA -> LITT RXEF010
- J1: value JST05_StepperMotor -> JST B5B-XH-A
- J6: value Conn_02x08_Top_Bottom -> 2x08 Edge Connector
- U4: value ATmega8A-A -> ATMEGA8A-AU
- Y1: value 16MHz -> 16,0000-HC49U-S
- moved C3 18.0 mm to (113.2, 110.2), turned to 0 degrees
- moved C4 16.9 mm to (113.2, 115.1), turned to 0 degrees
- moved Y1 4.58 mm to (117.6, 110.2), turned to -90 degrees
- moved C6 1.52 mm to (118.4, 105.7)
Routing:
- net +12V: track 45.9 -> 8.96 mm
- net GND: track 116.8 -> 88.2 mm
- net Net-(U4-PB6/XTAL1): track 17.9 -> 8.42 mm
- net Net-(J6-Pin_15): track 20.7 -> 16.6 mm
- net Net-(U4-ADC7): track 27.2 -> 25.3 mm
- net Net-(U4-PB7/XTAL2): track 11.4 -> 12.6 mm
- net /MOT_A: track 63.3 -> 64.4 mm
- net +5V: track 47.1 -> 48.2 mm
- net /BUS_TX: track 38.9 -> 39.8 mm
- net /BUS_RX: track 28.4 -> 28.9 mm
