File: hardware/module_controller/_autosave-ModuleController.kicad_sch (KiCad schematic)
At the start: 23 parts, among them J1 JST B5B-XH-A, J6 2x08 Edge Connector, U1 ULN2003, U2 A1101ELHL, U3 SN75176AP, U4 ATmega8A-A, Y1 16,0000-HC49U-S

Commit message: update schematics
Parts:
- F1: value RXEF010 -> LITT RXEF010
- U4: value ATmega8A-A -> ATMEGA8A-AU
Other:
- moved on the sheet: R2
Changed lines of the file:
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@@
 	(wire
 		(pts
+			(xy 115.57 85.09) (xy 115.57 91.44)
+		)
+		(stroke
+			(width 0)
+			(type default)
+		)
+	)
+	(wire
+		(pts
 			(xy 180.975 73.66) (xy 180.975 71.12)
 		)
@@
 	(wire
 		(pts
-			(xy 115.57 104.14) (xy 115.57 102.362)
+			(xy 115.57 104.14) (xy 115.57 99.06)
 		)
 		(stroke
@@
 	(wire
 		(pts
-			(xy 125.095 92.71) (xy 125.095 93.98)
+			(xy 125.095 92.71) (xy 125.095 113.03)
 		)
 		(stroke
@@
 	(symbol
 		(lib_id "power:+12V")
-		(at 115.57 94.742 0)
+		(at 115.57 85.09 0)
 		(mirror y)
 		(unit 1)
@@
 		(fields_autoplaced yes)
 		(property "Reference" "#PWR028"
-			(at 115.57 98.552 0)
+			(at 115.57 88.9 0)
 			(effects
 				(font
@@
 		)
 		(property "Value" "+12V"
-			(at 115.57 89.662 0)
+			(at 115.57 80.01 0)
 			(effects
 				(font
@@
 		)
 		(property "Footprint" ""
-			(at 115.57 94.742 0)
+			(at 115.57 85.09 0)
 			(effects
 				(font
@@
 		)
 		(property "Datasheet" ""
-			(at 115.57 94.742 0)
+			(at 115.57 85.09 0)
 			(effects
 				(font
@@
 		)
 		(property "Description" ""
-			(at 115.57 94.742 0)
+			(at 115.57 85.09 0)
 			(effects
 				(font
@@
 			)
 		)
-		(property "Value" "RXEF010"
+		(property "Value" "LITT RXEF010"
 			(at 70.485 183.515 0)
 			(effects
@@
 	(symbol
 		(lib_id "Device:R")
-		(at 115.57 98.552 0)
+		(at 115.57 95.25 0)
 		(unit 1)
 		(exclude_from_sim no)
@@
 		(fields_autoplaced yes)
 		(property "Reference" "R2"
-			(at 117.475 97.282 0)
+			(at 117.475 93.98 0)
 			(effects
 				(font
@@
 		)
 		(property "Value" "10k"
-			(at 117.475 99.822 0)
+			(at 117.475 96.52 0)
 			(effects
 				(font
@@
 		)
 		(property "Footprint" "Resistor_SMD:R_0805_2012Metric"
-			(at 113.792 98.552 90)
+			(at 113.792 95.25 90)
 			(effects
 				(font
@@
 		)
 		(property "Datasheet" "~"
-			(at 115.57 98.552 0)
+			(at 115.57 95.25 0)
 			(effects
 				(font
@@
 		)
 		(property "Description" ""
-			(at 115.57 98.552 0)
+			(at 115.57 95.25 0)
 			(effects
 				(font
@@
 		(fields_autoplaced yes)
 		(property "Reference" "U4"
-			(at 182.9309 71.12 0)
+			(at 183.1691 71.12 0)
 			(effects
 				(font
@@
 			)
 		)
-		(property "Value" "ATmega8A-A"
-			(at 182.9309 73.66 0)
+		(property "Value" "ATMEGA8A-AU"
+			(at 183.1691 73.66 0)
 			(effects
 				(font
@@
 	(symbol
 		(lib_id "power:GND")
-		(at 125.095 93.98 0)
+		(at 125.095 113.03 0)
 		(mirror y)
 		(unit 1)
@@
 		(fields_autoplaced yes)
 		(property "Reference" "#PWR015"
-			(at 125.095 100.33 0)
+			(at 125.095 119.38 0)
 			(effects
 				(font
@@
 		)
 		(property "Value" "GND"
-			(at 125.095 99.06 0)
+			(at 125.095 118.11 0)
 			(effects
 				(font
@@
 		)
 		(property "Footprint" ""
-			(at 125.095 93.98 0)
+			(at 125.095 113.03 0)
 			(effects
 				(font
@@
 		)
 		(property "Datasheet" ""
-			(at 125.095 93.98 0)
+			(at 125.095 113.03 0)
 			(effects
 				(font
@@
 		)
 		(property "Description" ""
-			(at 125.095 93.98 0)
+			(at 125.095 113.03 0)
 			(effects
 				(font
